File: Hardware/Circuits and PCB related/Sensor Cell with Comms/power.kicad_sch (KiCad schematic)
At the start: 15 parts, among them U4 TPS22950x, U5 TPS2421, U6 TPS2421

Commit message: Finished schematic, added all footprints, finishing ERC now to move onto the PCB planner to have Kicad do most of the heavy lifting
Parts:
- renumbered C7 to C13, C9 to C14, C10 to C15, C8 to C16, R12 to R23, R14 to R24, R8 to R25, R9 to R26, R11 to R27, R13 to R28, R10 to R29, R15 to R30, U4 to U10, U5 to U11, U6 to U9
Changed lines of the file:
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@@
 		(on_board yes)
 		(dnp no)
-		(property "Reference" "U5"
+		(property "Reference" "U11"
 			(at 83.82 44.958 0)
 			(effects
@@
 			(project "Sensor Cell with Comms"
 				(path "/953799b5-f11e-4770-941d-f5d23acc5c6d/fd73c0a6-9291-47e7-9fe4-221baafadf1c"
-					(reference "U5")
+					(reference "U11")
 					(unit 1)
 				)
@@
 		(dnp no)
 		(fields_autoplaced yes)
-		(property "Reference" "R15"
+		(property "Reference" "R30"
 			(at 115.57 73.6599 0)
 			(effects
@@
 			(project "Sensor Cell with Comms"
 				(path "/953799b5-f11e-4770-941d-f5d23acc5c6d/fd73c0a6-9291-47e7-9fe4-221baafadf1c"
-					(reference "R15")
+					(reference "R30")
 					(unit 1)
 				)
@@
 		(dnp no)
 		(fields_autoplaced yes)
-		(property "Reference" "#PWR018"
+		(property "Reference" "#PWR061"
 			(at 81.28 182.88 0)
 			(effects
@@
 			(project "Sensor Cell with Comms"
 				(path "/953799b5-f11e-4770-941d-f5d23acc5c6d/fd73c0a6-9291-47e7-9fe4-221baafadf1c"
-					(reference "#PWR018")
+					(reference "#PWR061")
 					(unit 1)
 				)
@@
 		(on_board yes)
 		(dnp no)
-		(property "Reference" "#PWR024"
+		(property "Reference" "#PWR062"
 			(at 91.44 81.28 0)
 			(effects
@@
 			(project "Sensor Cell with Comms"
 				(path "/953799b5-f11e-4770-941d-f5d23acc5c6d/fd73c0a6-9291-47e7-9fe4-221baafadf1c"
-					(reference "#PWR024")
+					(reference "#PWR062")
 					(unit 1)
 				)
@@
 		(dnp no)
 		(fields_autoplaced yes)
-		(property "Reference" "#PWR012"
+		(property "Reference" "#PWR055"
 			(at 52.07 161.29 0)
 			(effects
@@
 			(project "Sensor Cell with Comms"
 				(path "/953799b5-f11e-4770-941d-f5d23acc5c6d/fd73c0a6-9291-47e7-9fe4-221baafadf1c"
-					(reference "#PWR012")
+					(reference "#PWR055")
 					(unit 1)
 				)
@@
 		(on_board yes)
 		(dnp no)
-		(property "Reference" "#PWR020"
+		(property "Reference" "#PWR066"
 			(at 113.03 53.34 0)
 			(effects
@@
 			(project "Sensor Cell with Comms"
 				(path "/953799b5-f11e-4770-941d-f5d23acc5c6d/fd73c0a6-9291-47e7-9fe4-221baafadf1c"
-					(reference "#PWR020")
+					(reference "#PWR066")
 					(unit 1)
 				)
@@
 		(on_board yes)
 		(dnp no)
-		(property "Reference" "#PWR019"
+		(property "Reference" "#PWR063"
 			(at 93.98 148.59 0)
 			(effects
@@
 			(project "Sensor Cell with Comms"
 				(path "/953799b5-f11e-4770-941d-f5d23acc5c6d/fd73c0a6-9291-47e7-9fe4-221baafadf1c"
-					(reference "#PWR019")
+					(reference "#PWR063")
 					(unit 1)
 				)
@@
 		(dnp no)
 		(fields_autoplaced yes)
-		(property "Reference" "#PWR017"
+		(property "Reference" "#PWR056"
 			(at 58.42 173.99 0)
 			(effects
@@
 			(project "Sensor Cell with Comms"
 				(path "/953799b5-f11e-4770-941d-f5d23acc5c6d/fd73c0a6-9291-47e7-9fe4-221baafadf1c"
-					(reference "#PWR017")
+					(reference "#PWR056")
 					(unit 1)
 				)
@@
 		(on_board yes)
 		(dnp no)
-		(property "Reference" "#PWR023"
+		(property "Reference" "#PWR065"
 			(at 96.52 124.46 0)
 			(effects
@@
 			(project "Sensor Cell with Comms"
 				(path "/953799b5-f11e-4770-941d-f5d23acc5c6d/fd73c0a6-9291-47e7-9fe4-221baafadf1c"
-					(reference "#PWR023")
+					(reference "#PWR065")
 					(unit 1)
 				)
@@
 		(on_board yes)
 		(dnp no)
-		(property "Reference" "#PWR016"
+		(property "Reference" "#PWR057"
 			(at 59.69 143.51 0)
 			(effects
@@
 			(project "Sensor Cell with Comms"
 				(path "/953799b5-f11e-4770-941d-f5d23acc5c6d/fd73c0a6-9291-47e7-9fe4-221baafadf1c"
-					(reference "#PWR016")
+					(reference "#PWR057")
 					(unit 1)
 				)
@@
 		(dnp no)
 		(fields_autoplaced yes)
-		(property "Reference" "R13"
+		(property "Reference" "R28"
 			(at 99.06 123.1899 0)
 			(effects
@@
 			(project "Sensor Cell with Comms"
 				(path "/953799b5-f11e-4770-941d-f5d23acc5c6d/fd73c0a6-9291-47e7-9fe4-221baafadf1c"
-					(reference "R13")
+					(reference "R28")
 					(unit 1)
 				)
@@
 		(on_board yes)
 		(dnp no)
-		(property "Reference" "#PWR022"
+		(property "Reference" "#PWR059"
 			(at 74.93 129.54 0)
 			(effects
@@
 			(project "Sensor Cell with Comms"
 				(path "/953799b5-f11e-4770-941d-f5d23acc5c6d/fd73c0a6-9291-47e7-9fe4-221baafadf1c"
-					(reference "#PWR022")
+					(reference "#PWR059")
 					(unit 1)
 				)
@@
 		(on_board yes)
 		(dnp no)
-		(property "Reference" "C8"
+		(property "Reference" "C16"
 			(at 95.758 161.29 0)
 			(effects
@@
 			(project "Sensor Cell with Comms"
 				(path "/953799b5-f11e-4770-941d-f5d23acc5c6d/fd73c0a6-9291-47e7-9fe4-221baafadf1c"
-					(reference "C8")
+					(reference "C16")
 					(unit 1)
 				)
@@
 		(on_board yes)
 		(dnp no)
-		(property "Reference" "#PWR025"
+		(property "Reference" "#PWR067"
 			(at 113.03 74.93 0)
 			(effects
@@
 			(project "Sensor Cell with Comms"
 				(path "/953799b5-f11e-4770-941d-f5d23acc5c6d/fd73c0a6-9291-47e7-9fe4-221baafadf1c"
-					(reference "#PWR025")
+					(reference "#PWR067")
 					(unit 1)
 				)
@@
 		(dnp no)
 		(fields_autoplaced yes)
-		(property "Reference" "R8"
+		(property "Reference" "R25"
 			(at 83.82 167.6399 0)
 			(effects
@@
 			(project "Sensor Cell with Comms"
 				(path "/953799b5-f11e-4770-941d-f5d23acc5c6d/fd73c0a6-9291-47e7-9fe4-221baafadf1c"
-					(reference "R8")
+					(reference "R25")
 					(unit 1)
 				)
@@
 		(on_board yes)
 		(dnp no)
-		(property "Reference" "C7"
+		(property "Reference" "C13"
 			(at 52.832 161.29 0)
 			(effects
@@
 			(project "Sensor Cell with Comms"
 				(path "/953799b5-f11e-4770-941d-f5d23acc5c6d/fd73c0a6-9291-47e7-9fe4-221baafadf1c"
-					(reference "C7")
+					(reference "C13")
 					(unit 1)
 				)
@@
 		(on_board yes)
 		(dnp no)
-		(property "Reference" "#PWR015"
+		(property "Reference" "#PWR060"
 			(at 76.2 95.25 0)
 			(effects
@@
 			(project "Sensor Cell with Comms"
 				(path "/953799b5-f11e-4770-941d-f5d23acc5c6d/fd73c0a6-9291-47e7-9fe4-221baafadf1c"
-					(reference "#PWR015")
+					(reference "#PWR060")
 					(unit 1)
 				)
@@
 		(on_board yes)
 		(dnp no)
-		(property "Reference" "R12"
+		(property "Reference" "R23"
 			(at 65.786 128.778 0)
 			(effects
@@
 			(project "Sensor Cell with Comms"
 				(path "/953799b5-f11e-4770-941d-f5d23acc5c6d/fd73c0a6-9291-47e7-9fe4-221baafadf1c"
-					(reference "R12")
+					(reference "R23")
 					(unit 1)
 				)
@@
 		(dnp no)
 		(fields_autoplaced yes)
-		(property "Reference" "#PWR013"
+		(property "Reference" "#PWR054"
 			(at 44.45 110.49 0)
 			(effects
@@
 			(project "Sensor Cell with Comms"
 				(path "/953799b5-f11e-4770-941d-f5d23acc5c6d/fd73c0a6-9291-47e7-9fe4-221baafadf1c"
-					(reference "#PWR013")
+					(reference "#PWR054")
 					(unit 1)
 				)
@@
 		(dnp no)
 		(fields_autoplaced yes)
-		(property "Reference" "#PWR014"
+		(property "Reference" "#PWR058"
 			(at 60.96 62.23 0)
 			(effects
@@
 			(project "Sensor Cell with Comms"
 				(path "/953799b5-f11e-4770-941d-f5d23acc5c6d/fd73c0a6-9291-47e7-9fe4-221baafadf1c"
-					(reference "#PWR014")
+					(reference "#PWR058")
 					(unit 1)
 				)
@@
 		(on_board yes)
 		(dnp no)
-		(property "Reference" "U6"
+		(property "Reference" "U9"
 			(at 67.31 93.218 0)
 			(effects
@@
 			(project "Sensor Cell with Comms"
 				(path "/953799b5-f11e-4770-941d-f5d23acc5c6d/fd73c0a6-9291-47e7-9fe4-221baafadf1c"
-					(reference "U6")
+					(reference "U9")
 					(unit 1)
 				)
@@
 		(on_board yes)
 		(dnp no)
-		(property "Reference" "R14"
+		(property "Reference" "R24"
 			(at 81.534 80.518 0)
 			(effects
@@
 			(project "Sensor Cell with Comms"
 				(path "/953799b5-f11e-4770-941d-f5d23acc5c6d/fd73c0a6-9291-47e7-9fe4-221baafadf1c"
-					(reference "R14")
+					(reference "R24")
 					(unit 1)
 				)
@@
 		(on_board yes)
 		(dnp no)
-		(property "Reference" "C9"
+		(property "Reference" "C14"
 			(at 70.104 134.62 0)
 			(effects
@@
 			(project "Sensor Cell with Comms"
 				(path "/953799b5-f11e-4770-941d-f5d23acc5c6d/fd73c0a6-9291-47e7-9fe4-221baafadf1c"
-					(reference "C9")
+					(reference "C14")
 					(unit 1)
 				)
@@
 		(on_board yes)
 		(dnp no)
-		(property "Reference" "C10"
+		(property "Reference" "C15"
 			(at 86.614 86.36 0)
 			(effects
@@
 			(project "Sensor Cell with Comms"
 				(path "/953799b5-f11e-4770-941d-f5d23acc5c6d/fd73c0a6-9291-47e7-9fe4-221baafadf1c"
-					(reference "C10")
+					(reference "C15")
 					(unit 1)
 				)
@@
 		(dnp no)
 		(fields_autoplaced yes)
-		(property "Reference" "R10"
+		(property "Reference" "R29"
 			(at 115.57 52.0699 0)
 			(effects
@@
 			(project "Sensor Cell with Comms"
 				(path "/953799b5-f11e-4770-941d-f5d23acc5c6d/fd73c0a6-9291-47e7-9fe4-221baafadf1c"
-					(reference "R10")
+					(reference "R29")
 					(unit 1)
 				)
@@
 		(dnp no)
 		(fields_autoplaced yes)
-		(property "Reference" "R9"
+		(property "Reference" "R26"
 			(at 96.52 147.3199 0)
 			(effects
@@
 			(project "Sensor Cell with Comms"
 				(path "/953799b5-f11e-4770-941d-f5d23acc5c6d/fd73c0a6-9291-47e7-9fe4-221baafadf1c"
-					(reference "R9")
+					(reference "R26")
 					(unit 1)
 				)
@@
 		(on_board yes)
 		(dnp no)
-		(property "Reference" "#PWR021"
+		(property "Reference" "#PWR064"
 			(at 96.52 101.6 0)
 			(effects
@@
 			(project "Sensor Cell with Comms"
 				(path "/953799b5-f11e-4770-941d-f5d23acc5c6d/fd73c0a6-9291-47e7-9fe4-221baafadf1c"
-					(reference "#PWR021")
+					(reference "#PWR064")
 					(unit 1)
 				)
@@
 		(dnp no)
 		(fields_autoplaced yes)
-		(property "Reference" "U4"
+		(property "Reference" "U10"
 			(at 70.485 144.78 0)
 			(effects
@@
 			(project "Sensor Cell with Comms"
 				(path "/953799b5-f11e-4770-941d-f5d23acc5c6d/fd73c0a6-9291-47e7-9fe4-221baafadf1c"
-					(reference "U4")
+					(reference "U10")
 					(unit 1)
 				)
@@
 		(dnp no)
 		(fields_autoplaced yes)
-		(property "Reference" "R11"
+		(property "Reference" "R27"
 			(at 99.06 100.3299 0)
 			(effects
@@
 			(project "Sensor Cell with Comms"
 				(path "/953799b5-f11e-4770-941d-f5d23acc5c6d/fd73c0a6-9291-47e7-9fe4-221baafadf1c"
-					(reference "R11")
-					(unit 1)
-				)
+					(reference "R27")
+					(unit 1)
+				)

Commit message: First revision of PCB nearly done, Need to finish up 1v8 planes then wire components together
Parts:
- added C18, C19, C20, C21: 10u, Capacitor_SMD:C_0603_1608Metric_Pad1.08x0.95mm_HandSolder, symbol Device:C
- R25: value 530 -> 630
Connections:
- net +3V3DC: now also C20.2
- net +3V3_railMonitor: now also C18.2
- net +5V0DC: now also C21.2
- net +5V0_railMonitor: now also C19.2
- net GND: now also C18.1, C19.1, C20.1, C21.1
Other:
- title: (none) -> Power eFuses
