File: Hardware/Circuits and PCB related/Sensor Cell with Comms Rev2/Sensor Cell with Comms.kicad_sch (KiCad schematic)
At the start: 27 parts, among them J1 MolexMicroFit3_1, J2 MolexMicroFit3_2, J3 MolexMicroFit3_3, U1 STM32F103C6T6

Commit message: Found a GUI driven code tool, lets me configure every pin via a GUI and now we just need to write the logical steps of what signals do what. Need to Re-add the MCP2518 open source driver since I deleted the entire old code for my STM as it kept bringing errors due to my misconfigurations
Connections:
- net GND: now also C22.2; no longer C22.1
- net at JP1.1 (A), U1.24 (VDD): now also C22.1; no longer C22.2
Other:
- moved on the sheet: C22
